File: Hardware/Compresseur_KiCad/Compresseur.kicad_sch (KiCad schematic)
At the start: 0 parts

Commit message: Add files via upload
Parts:
- added R6 (x2): PTV09A-4020F-B103, PTV09A4020FB103, symbol PTV09A-4020F-B103:PTV09A-4020F-B103
Connections:
- new net 3V3: R6.3, R6.3
- new net Earth: R6.4 (MH1), R6.4 (MH1), R6.5 (MH2), R6.5 (MH2)
- new net Filter1: R6.2
- new net Filter2: R6.2
- new net GND: R6.1, R6.1
Other:
- added sheet Codec Audio (Codec.kicad_sch)

Commit message: Add files via upload
Parts:
- added U3: ~, symbol Driver_Display:Oled_screen
Connections:
- net 3V3: now also U3.1 (VCC)
- net GND: now also U3.2 (GND)
- new net SCL_Nucleo: U3.3 (SCL)
- new net SDA_Nucleo: U3.4 (SDA)
Changed lines of the file:
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@@
+    (stroke (width 0) (type default))
+  )
+  (wire (pts (xy 227.33 116.84) (xy 227.33 121.92))
+    (stroke (width 0) (type default))
+  )
+  (wire (pts (xy 240.03 116.84) (xy 240.03 121.92))
+    (stroke (width 0) (type default))
+  )
+  (wire (pts (xy 236.22 116.84) (xy 236.22 121.92))
     (stroke (width 0) (type default))
   )
@@
     (stroke (width 0) (type default))
   )
+  (wire (pts (xy 231.14 116.84) (xy 231.14 121.92))
+    (stroke (width 0) (type default))
+  )
   (wire (pts (xy 97.79 121.92) (xy 97.79 127))
     (stroke (width 0) (type default))
@@
     (stroke (width 0) (type default))
   )
+  (global_label "3V3" (shape input) (at 231.14 121.92 270) (fields_autoplaced)
+    (effects (font (size 1.27 1.27)) (justify right))
+    (property "Intersheetrefs" "${INTERSHEET_REFS}" (at 231.14 128.4128 90)
+      (effects (font (size 1.27 1.27)) (justify right) hide)
+    )
+  )
   (global_label "GND" (shape input) (at 177.8 90.17 0) (fields_autoplaced)
     (effects (font (size 1.27 1.27)) (justify left))
@@
     )
   )
+  (global_label "SCL_Nucleo" (shape input) (at 236.22 121.92 270) (fields_autoplaced)
+    (effects (font (size 1.27 1.27)) (justify right))
+    (property "Intersheetrefs" "${INTERSHEET_REFS}" (at 236.22 135.8513 90)
+      (effects (font (size 1.27 1.27)) (justify right) hide)
+    )
+  )
   (global_label "GND" (shape input) (at 99.06 91.44 0) (fields_autoplaced)
     (effects (font (size 1.27 1.27)) (justify left))
@@
     (effects (font (size 1.27 1.27)) (justify right))
     (property "Intersheetrefs" "${INTERSHEET_REFS}" (at 87.4872 91.44 0)
+      (effects (font (size 1.27 1.27)) (justify right) hide)
+    )
+  )
+  (global_label "GND" (shape input) (at 227.33 121.92 270) (fields_autoplaced)
+    (effects (font (size 1.27 1.27)) (justify right))
+    (property "Intersheetrefs" "${INTERSHEET_REFS}" (at 227.33 128.7757 90)
+      (effects (font (size 1.27 1.27)) (justify right) hide)
+    )
+  )
+  (global_label "SDA_Nucleo" (shape input) (at 240.03 121.92 270) (fields_autoplaced)
+    (effects (font (size 1.27 1.27)) (justify right))
+    (property "Intersheetrefs" "${INTERSHEET_REFS}" (at 240.03 135.9118 90)
       (effects (font (size 1.27 1.27)) (justify right) hide)
     )
@@
         )
       )
+    )
+  )
+  (symbol (lib_id "Driver_Display:Oled_screen") (at 233.68 99.06 0) (unit 1)
+    (in_bom yes) (on_board yes) (dnp no) (fields_autoplaced)
+    (property "Reference" "U3" (at 243.84 107.315 0)
+      (effects (font (size 1.27 1.27)) (justify left))
+    )
+    (property "Value" "~" (at 233.68 99.06 0)
+      (effects (font (size 1.27 1.27)))
+    )
+    (property "Footprint" "" (at 233.68 99.06 0)
+      (effects (font (size 1.27 1.27)) hide)
+    )
+    (property "Datasheet" "" (at 233.68 99.06 0)
+      (effects (font (size 1.27 1.27)) hide)
+    )
+    (pin "3")
+    (pin "1")
+    (pin "2")
+    (pin "4")
+    (instances
+      (project "Compresseur"
+        (path "/c9f90ba6-9ce8-4fd1-ae7a-2fb80556f20b"
+          (reference "U3") (unit 1)
+        )
+      )
